Commit message: rviz functioning well now

File: open_manipulator_pro/open_manipulator_pro_description/urdf/open_manipulator_pro.gazebo.xacro (robot description, xacro)
@@ -27,15 +27,11 @@
   <RefLink ref="link5"/>
   <!-- gripper_link -->
-  <RefLink ref="gripper_link"/>
+  <RefLink ref="link6"/>
   <!-- gripper_link_sub -->
-  <RefLink ref="gripper_link_sub"/>
-  <!-- end effector link -->
-  <gazebo reference="end_effector_link">
-    <material>Gazebo/Red</material>
-  </gazebo>
+  <RefLink ref="end_link"/>
   <!-- ros_control plugin -->
   <gazebo>
     <plugin name="gazebo_ros_control" filename="libgazebo_ros_control.so">
-      <robotNamespace>open_manipulator_x</robotNamespace>
+      <robotNamespace>open_manipulator_pro</robotNamespace>
       <controlPeriod>0.001</controlPeriod>
       <robotSimType>gazebo_ros_control/DefaultRobotHWSim</robotSimType>

File: open_manipulator_pro/open_manipulator_pro_description/urdf/open_manipulator_pro.urdf.xacro (robot description, xacro)
@@ -2,4 +2,6 @@
 <!-- OpenManipulator Chain -->
 <robot name="open_manipulator_pro" xmlns:xacro="http://ros.org/wiki/xacro">
+  <!-- some parameters -->
+  <!-- <xacro:property name="pi" value="3.141592654" /> -->
   <!-- Import all Gazebo-customization elements, including Gazebo colors -->
   <xacro:include filename="$(find open_manipulator_pro_description)/urdf/open_manipulator_pro.gazebo.xacro" />
@@ -61,17 +63,17 @@
   <!-- link 1 -->
   <link name="link1">
-    <collision>
-      <origin xyz="0 0 0" rpy="0 0 0"/>
-      <geometry>
-        <mesh filename="package://open_manipulator_pro_description/meshes/link_1.stl" scale="0.001 0.001 0.001"/>
-      </geometry>
-    </collision>
-    <visual>
-      <origin xyz="0 0 0" rpy="0 0 0"/>
-      <geometry>
-        <mesh filename="package://open_manipulator_pro_description/meshes/link_1.stl" scale="0.001 0.001 0.001"/>
-      </geometry>
-      <material name="grey"/>
-    </visual>
+    <visual>
+      <origin xyz="0 0 0" rpy="0 0 0"/>
+      <geometry>
+        <mesh filename="package://open_manipulator_pro_description/meshes/link1.stl" scale="0.001 0.001 0.001"/>
+      </geometry>
+      <material name="grey"/>
+    </visual>
+    <collision>
+      <origin xyz="0 0 0" rpy="0 0 0"/>
+      <geometry>
+        <mesh filename="package://open_manipulator_pro_description/meshes/link1.stl" scale="0.001 0.001 0.001"/>
+      </geometry>
+    </collision>
     <inertial>
       <origin xyz="0.00023 0.00000 0.06223" rpy="0 0 0"/>
@@ -87,5 +89,5 @@
     <origin xyz="0.0 0.0 0.126" rpy="0 0 0"/>
     <axis xyz="0 0 1"/>
-    <limit velocity="6.5" effort="1000" lower="${-pi*0.5}" upper="${pi*0.5}" />
+    <limit velocity="6.5" effort="1000" lower="-1.57079632679" upper="1.57079632679" />
     <dynamics damping="0.7"/>
   </joint>
@@ -94,17 +96,17 @@
   <!-- link 2 -->
   <link name="link2">
-    <collision>
-      <origin xyz="0 0 0" rpy="0 0 0"/>
-      <geometry>
-        <mesh filename="package://open_manipulator_pro_description/meshes/link_2.stl" scale="0.001 0.001 0.001"/>
-      </geometry>
-    </collision>
-    <visual>
-      <origin xyz="0 0 0" rpy="0 0 0"/>
-      <geometry>
-        <mesh filename="package://open_manipulator_pro_description/meshes/link_2.stl" scale="0.001 0.001 0.001"/>
-      </geometry>
-      <material name="grey"/>
-    </visual>
+    <visual>
+      <origin xyz="0 0 0" rpy="0 0 0"/>
+      <geometry>
+        <mesh filename="package://open_manipulator_pro_description/meshes/link2.stl" scale="0.001 0.001 0.001"/>
+      </geometry>
+      <material name="grey"/>
+    </visual>
+    <collision>
+      <origin xyz="0 0 0" rpy="0 0 0"/>
+      <geometry>
+        <mesh filename="package://open_manipulator_pro_description/meshes/link2.stl" scale="0.001 0.001 0.001"/>
+      </geometry>
+    </collision>
     <inertial>
       <origin xyz="0.00000 0.00080 0.03183" rpy="0 0 0"/>
@@ -121,5 +123,5 @@
     <origin xyz="0.0 0.0 0.033" rpy="0 0 0"/>
     <axis xyz="0 1 0"/>
-    <limit velocity="6.5" effort="1000" lower="${-pi*0.5}" upper="${pi*0.5}" />
+    <limit velocity="6.5" effort="1000" lower="-1.57079632679" upper="1.57079632679" />
     <dynamics damping="0.7"/>
   </joint>
@@ -128,17 +130,17 @@
   <!-- link 3 -->
   <link name="link3">
-    <collision>
+    <visual>
       <origin xyz="0 0.069 0" rpy="0 0 0"/>
       <geometry>
-        <mesh filename="package://open_manipulator_pro_description/meshes/link_3.stl" scale="0.001 0.001 0.001"/>
-      </geometry>
-    </collision>
-    <visual>
+        <mesh filename="package://open_manipulator_pro_description/meshes/link3.stl" scale="0.001 0.001 0.001"/>
+      </geometry>
+      <material name="grey"/>
+    </visual>
+    <collision>
       <origin xyz="0 0.069 0" rpy="0 0 0"/>
       <geometry>
-        <mesh filename="package://open_manipulator_pro_description/meshes/link_3.stl" scale="0.001 0.001 0.001"/>
-      </geometry>
-      <material name="grey"/>
-    </visual>
+        <mesh filename="package://open_manipulator_pro_description/meshes/link3.stl" scale="0.001 0.001 0.001"/>
+      </geometry>
+    </collision>
     <inertial>
       <origin xyz="0.01768 0.00019 0.20524" rpy="0 0 0"/>
@@ -154,5 +156,5 @@
     <origin xyz="0.03000 0.0 0.26400" rpy="0 0 0"/>
     <axis xyz="0 1 0"/>
-    <limit velocity="6.5" effort="1000" lower="${-pi*0.5}" upper="${pi*0.5}" />
+    <limit velocity="6.5" effort="1000" lower="-1.57079632679" upper="1.57079632679" />
     <dynamics damping="0.7"/>
   </joint>
@@ -161,17 +163,17 @@
   <!-- link 4 -->
   <link name="link4">
-    <collision>
+    <visual>
       <origin xyz="0 0.05750 0" rpy="0 0 0"/>
       <geometry>
-        <mesh filename="package://open_manipulator_pro_description/meshes/link_4.stl" scale="0.001 0.001 0.001"/>
-      </geometry>
-    </collision>
-    <visual>
+        <mesh filename="package://open_manipulator_pro_description/meshes/link4.stl" scale="0.001 0.001 0.001"/>
+      </geometry>
+      <material name="grey"/>
+    </visual>
+    <collision>
       <origin xyz="0 0.05750 0" rpy="0 0 0"/>
       <geometry>
-        <mesh filename="package://open_manipulator_pro_description/meshes/link_4.stl" scale="0.001 0.001 0.001"/>
-      </geometry>
-      <material name="grey"/>
-    </visual>
+        <mesh filename="package://open_manipulator_pro_description/meshes/link4.stl" scale="0.001 0.001 0.001"/>
+      </geometry>
+    </collision>
     <inertial>
       <origin xyz="-0.07025 0.00034 -0.00021" rpy="0 0 0"/>
@@ -187,5 +189,5 @@
     <origin xyz="0.19500 0.0 0.03000" rpy="0 0 0"/>
     <axis xyz="1 0 0"/>
-    <limit velocity="6.5" effort="1000" lower="${-pi*0.5}" upper="${pi*0.5}" />
+    <limit velocity="6.5" effort="1000" lower="-1.57079632679" upper="1.57079632679" />
     <dynamics damping="0.7"/>
   </joint>
@@ -194,17 +196,17 @@
   <!-- link 5 -->
   <link name="link5">
-    <collision>
-      <origin xyz="0 0 0" rpy="0 0 0"/>
-      <geometry>
-        <mesh filename="package://open_manipulator_pro_description/meshes/link_5.stl" scale="0.001 0.001 0.001"/>
-      </geometry>
-    </collision>
-    <visual>
-      <origin xyz="0 0 0" rpy="0 0 0"/>
-      <geometry>
-        <mesh filename="package://open_manipulator_pro_description/meshes/link_5.stl" scale="0.001 0.001 0.001"/>
-      </geometry>
-      <material name="grey"/>
-    </visual>
+    <visual>
+      <origin xyz="0 0 0" rpy="0 0 0"/>
+      <geometry>
+        <mesh filename="package://open_manipulator_pro_description/meshes/link5.stl" scale="0.001 0.001 0.001"/>
+      </geometry>
+      <material name="grey"/>
+    </visual>
+    <collision>
+      <origin xyz="0 0 0" rpy="0 0 0"/>
+      <geometry>
+        <mesh filename="package://open_manipulator_pro_description/meshes/link5.stl" scale="0.001 0.001 0.001"/>
+      </geometry>
+    </collision>
     <inertial>
       <origin xyz="0.05642 -0.00217 0.00002" rpy="0 0 0"/>
@@ -221,5 +223,5 @@
     <origin xyz="0.06300 0.00 0.00000" rpy="0 0 0"/>
     <axis xyz="0 1 0"/>
-    <limit velocity="6.5" effort="1000" lower="${-pi*0.5}" upper="${pi*0.5}" />
+    <limit velocity="6.5" effort="1000" lower="-1.57079632679" upper="1.57079632679" />
     <dynamics damping="0.7"/>
   </joint>
@@ -228,17 +230,17 @@
   <!-- link 6 -->
   <link name="link6">
-    <collision>
+    <visual>
       <origin xyz="0 0.04500 0" rpy="0 0 0"/>
       <geometry>
-        <mesh filename="package://open_manipulator_pro_description/meshes/link_6.stl" scale="0.001 0.001 0.001"/>
-      </geometry>
-    </collision>
-    <visual>
+        <mesh filename="package://open_manipulator_pro_description/meshes/link6.stl" scale="0.001 0.001 0.001"/>
+      </geometry>
+      <material name="grey"/>
+    </visual>
+    <collision>
       <origin xyz="0 0.04500 0" rpy="0 0 0"/>
       <geometry>
-        <mesh filename="package://open_manipulator_pro_description/meshes/link_6.stl" scale="0.001 0.001 0.001"/>
-      </geometry>
-      <material name="grey"/>
-    </visual>
+        <mesh filename="package://open_manipulator_pro_description/meshes/link6.stl" scale="0.001 0.001 0.001"/>
+      </geometry>
+    </collision>
     <inertial>
       <!-- <origin xyz="0.06831 -0.04457 0.00000" rpy="0 0 0"/> -->
@@ -255,5 +257,5 @@
     <origin xyz="0.12300 0.000 0.00000" rpy="0 0 0"/>
     <axis xyz="1 0 0"/>
-    <limit velocity="6.5" effort="1000" lower="${-pi*0.5}" upper="${pi*0.5}" />
+    <limit velocity="6.5" effort="1000" lower="-1.57079632679" upper="1.57079632679" />
     <dynamics damping="0.7"/>
   </joint>
@@ -262,17 +264,17 @@
   <!-- end link -->
   <link name="end_link">
-    <collision>
+    <visual>
       <origin xyz="0 0 0" rpy="0 0 0"/>
       <geometry>
         <mesh filename="package://open_manipulator_pro_description/meshes/end_link.stl" scale="0.001 0.001 0.001"/>
       </geometry>
-    </collision>
-    <visual>
+      <material name="grey"/>
+    </visual>
+    <collision>
       <origin xyz="0 0 0" rpy="0 0 0"/>
       <geometry>
         <mesh filename="package://open_manipulator_pro_description/meshes/end_link.stl" scale="0.001 0.001 0.001"/>
       </geometry>
-      <material name="grey"/>
-    </visual>
+    </collision>
     <inertial>
       <origin xyz="0.00337 0.00000 0.00000" rpy="0 0 0"/>
